File: Pure LFO.sch (EAGLE design)
At the start: 46 parts, among them T3 TRANS_PAIR, U1 DUAL_OPAMP, U2 QUAD_OPAMP

Commit message: LFO 2.1
Parts:
- removed L1, L2, L3: LED_RG_SMD_REV, INSTRUO:LED_RG_SMD_REV
- removed R16: 15K, rcl:R-US_R0805
- removed R18: 50K, rcl:R-US_R0805
- removed R19: 20K, rcl:R-US_R0805
- removed R20, R21, R22: 2K*, rcl:R-US_R0805
- removed U1: DUAL_OPAMP, INSTRUO:DUAL_OPAMP
- removed U2: QUAD_OPAMP, INSTRUO:QUAD_OPAMP
- added IC1: TL074, GMSN:OPAMP_QUADD
- added IC2: TL072, GMSN:OPAMP_QUADD
- C1: value 47nF -> 5n1F; device rcl:C-USC0805K -> GMSN:CAPACITOR-USC0805
- C2, C3: value 10u -> 10uF; device rcl:CPOL-US153CLV-0505 -> GMSN:CAPACITOR_POL-US153CLV-0505
- C4, C5, C7, C8: value 0.1u -> 100nF; device rcl:C-USC0805K -> GMSN:CAPACITOR-USC0805
- C6: device rcl:C-USC0805K -> GMSN:CAPACITOR-USC0805
- D1, D2: value (none) -> STTH102A; device adafruit:DIODESMA -> GMSN:DIODESMA
- JP1: value M05X2SHD -> HEADER2X5SHD; device SparkFun-Connectors:M05X2SHD -> GMSN:HEADER2X5SHD
- R1: value 1K -> 100R; device rcl:R-US_R0805 -> GMSN:RESISTOR_USR0805
- R10, R12, R14, R15, R17, R9: value 10K -> 10k; device rcl:R-US_R0805 -> GMSN:RESISTOR_USR0805
- R11: value 400R -> 402R; device rcl:R-US_R0805 -> GMSN:RESISTOR_USR0805
- R13, R8: value 2K -> 2k; device rcl:R-US_R0805 -> GMSN:RESISTOR_USR0805
- R2: value 300R? -> 3M3; device rcl:R-US_R0805 -> GMSN:RESISTOR_USR0805
- R3: value 3M -> 3k3; device rcl:R-US_R0805 -> GMSN:RESISTOR_USR0805
- R4: value 12K -> 12k; device rcl:R-US_R0805 -> GMSN:RESISTOR_USR0805
- R5: value 33K -> 33k; device rcl:R-US_R0805 -> GMSN:RESISTOR_USR0805
- R6: value 1K3 -> 1k3; device rcl:R-US_R0805 -> GMSN:RESISTOR_USR0805
- R7: value 3K3 -> 3k3; device rcl:R-US_R0805 -> GMSN:RESISTOR_USR0805
- RATE: value B100K -> B100k; device INSTRUO:Q-POT -> GMSN:RESISTOR_VARIABLE9MM_POT
- RATESW: value TOGGLE_ON_OFF_ON -> SWITCH_TOGGLE_SPDT; device INSTRUO:TOGGLE_ON_OFF_ON -> GMSN:SWITCH_TOGGLE_SPDT
- SINE_OUT, SQU_OUT, TRI_OUT: value S_JACK -> SOCKET_MONO_3.5MMPJ301M-12; device INSTRUO:S_JACK -> GMSN:SOCKET_MONO_3.5MMPJ301M-12
- T3: value TRANS_PAIR -> DMMT3904W-7-F; device QuBit:TRANS_PAIR -> GMSN:TRANSISTOR_PAIR_NPN
- TR1: value 100K -> 100k; device INSTRUO:TRIM_3269W -> GMSN:RESISTOR_VARIABLETRIMMER_TH
- TR2: device INSTRUO:TRIM_3269W -> GMSN:RESISTOR_VARIABLETRIMMER_TH
Connections:
- removed net L_SIN: R21.2, SINE_OUT.NORM
- removed net L_SQU: R20.2, SQU_OUT.NORM
- removed net L_TRI: R22.2, TRI_OUT.NORM
- removed net N$13: L1G$1.C, L1G$2.A, L2G$1.C, L2G$2.A, L3G$1.C, L3G$2.A, R18.1, R5.1, RATE.3, U2G$4.OUT
- removed net N$15: L1G$1.A, L1G$2.C, R22.1
- removed net N$16: L2G$1.A, L2G$2.C, R21.1
- removed net N$17: L3G$1.A, L3G$2.C, R20.1
- removed net SINE: R17.1, SINE_OUT.TIP, U1G$1.OUT
- new net SINE_WAVE: IC1C.+IN, IC2A.OUT, R17.1
- new net SQUARE_WAVE: IC1D.OUT, IC2C.+IN, R5.1, RATE.3
- new net TRIANGLE_WAVE: C1.2, IC1B.OUT, IC2D.+IN, R4.2, R6.2
- net +12V: now also IC1P.V+, IC2P.V+; no longer U1G$3.+12V, U2G$5.+12V
- net -12V: now also IC1P.V-, IC2P.V-; no longer U1G$4.-12V, U2G$6.-12V
- net GND: now also IC1B.+IN, IC1D.-IN, SINE_OUT.SLEEVE, SQU_OUT.SLEEVE, TRI_OUT.SLEEVE; no longer R16.1, R19.1, SINE_OUT.GND, SQU_OUT.GND, TRI_OUT.GND, U2G$2.+IN, U2G$4.-IN
- net N$32: now also IC2B.-IN; no longer U1G$2.-IN
- net N$33: now also IC1A.-IN, IC1A.OUT; no longer U2G$1.-IN, U2G$1.OUT
- net N$34: now also IC2B.+IN; no longer U1G$2.+IN
- net N$35: now also IC1A.+IN; no longer U2G$1.+IN
- net N$38: now also IC2A.-IN; no longer R16.2, U1G$1.-IN
- net N$5: now also IC2C.-IN, IC2C.OUT, SQU_OUT.TIP; no longer R18.2, R19.2, U2G$3.+IN
- net N$6: now also IC1B.-IN; no longer U2G$2.-IN
- net N$7: now also IC2D.-IN, IC2D.OUT; no longer C1.2, R4.2, R6.2, U2G$2.OUT
- net N$8: now also IC1C.-IN, IC1C.OUT, SINE_OUT.TIP; no longer SQU_OUT.TIP, U2G$3.-IN, U2G$3.OUT
- net N$9: now also IC1D.+IN; no longer U2G$4.+IN
- net SINE_PRE: now also IC2A.+IN, IC2B.OUT; no longer U1G$1.+IN, U1G$2.OUT

Commit message: LFO 2.2
LFO Updated to V2.2 20/4/21

Traces rerouted.
Schmitt Trigger error corrected.
Connections:
- removed net N$38: IC2A.-IN, R17.2
- new net N$10: IC2C.-IN, IC2C.OUT, R17.2
- net GND: now also IC1C.+IN; no longer IC1B.+IN
- net N$33: now also IC1B.-IN, IC1B.OUT; no longer IC1A.-IN, IC1A.OUT
- net N$35: now also IC1B.+IN; no longer IC1A.+IN
- net N$5: now also IC1A.-IN, IC1A.OUT; no longer IC2C.-IN, IC2C.OUT
- net N$6: now also IC1C.-IN; no longer IC1B.-IN
- net N$7: now also IC2A.-IN, IC2A.OUT; no longer IC2D.-IN, IC2D.OUT
- net N$8: now also IC2D.-IN, IC2D.OUT; no longer IC1C.-IN, IC1C.OUT
- net SINE_PRE: now also IC2C.+IN; no longer IC2A.+IN
- net SINE_WAVE: now also IC2D.+IN; no longer IC1C.+IN, IC2A.OUT
- net SQUARE_WAVE: now also IC1A.+IN; no longer IC2C.+IN
- net TRIANGLE_WAVE: now also IC1C.OUT, IC2A.+IN; no longer IC1B.OUT, IC2D.+IN
